Commit message: nav2 basic tutorial robot added

File: src/basic_mobile_robot/src/description/basic_mobile_bot_v1.urdf.xacro (robot description, xacro)
@@ -18,5 +18,5 @@
   <!-- Position the caster wheel along the x-axis -->
   <xacro:property name="caster_xoff" value="0.217"/>
-  <!-- Define intertial property macros  -->
+  <!-- Define inertial property macros  -->
   <xacro:macro name="box_inertia" params="m w h d">
     <inertial>
@@ -53,5 +53,5 @@
       <origin xyz="0 0 -0.05" rpy="1.5707963267949 0 3.141592654"/>
       <geometry>
-        <mesh filename="package://basic_mobile_robot/meshes/robot_base.stl" />
+        <mesh filename="package://basic_mobile_robot/meshes/basic_mobile_robot/robot_base.stl" />
       </geometry>
       <material name="Red">
